File: Phase_B/Arduino_uno_Shield/Arduino_uno_Shield.kicad_sch (KiCad schematic)
At the start: 20 parts, among them J1 Power, J2 Digital/PWM, J3 Analog, J4 Digital/PWM, J5 CONN_GYRO, J6 Conn_01x04, J7 Temp_Digital, SW1 SW_DPST_x2, SW2 SW_DPST_x2, SW3 SW_DPST_x2, SW4 SW_DPST_x2, SW6 SW_DPST_x2

Commit message: Phase_B
Parts:
- removed J5: CONN_GYRO, Connector_PinSocket_2.54mm:PinSocket_1x08_P2.54mm_Vertical, symbol Connector_Generic:Conn_01x08
- removed J6: Conn_01x04, Connector_PinSocket_2.54mm:PinSocket_1x04_P2.54mm_Vertical, symbol Connector_Generic:Conn_01x04
- removed J7: Temp_Digital, Connector_JST:JST_XH_B3B-XH-A_1x03_P2.50mm_Vertical, symbol Connector_Generic:Conn_01x03
- removed R1, R2, R3, R4, R5, R6: R, Resistor_THT:R_Axial_DIN0207_L6.3mm_D2.5mm_P10.16mm_Horizontal, symbol Device:R
- removed SW1, SW2, SW3, SW4, SW6: SW_DPST_x2, Button_Switch_THT:SW_PUSH_6mm, symbol Switch:SW_DPST_x2
- added J10: CONN_DISPLAY, Connector_PinSocket_2.54mm:PinSocket_1x04_P2.54mm_Vertical, symbol Connector_Generic:Conn_01x04
- added J11: Temp_Digital, Connector_JST:JST_XH_B3B-XH-A_1x03_P2.50mm_Vertical, symbol Connector_Generic:Conn_01x03
- added J9: CONN_GYRO, Connector_PinSocket_2.54mm:PinSocket_1x08_P2.54mm_Vertical, symbol Connector_Generic:Conn_01x08
- added R1: 1k, Resistor_THT:R_Axial_DIN0207_L6.3mm_D2.5mm_P10.16mm_Horizontal, symbol Device:R_Small
- added R2, R3, R4, R5, R6: 100k, Resistor_THT:R_Axial_DIN0207_L6.3mm_D2.5mm_P10.16mm_Horizontal, symbol Device:R_Small
- added SW1, SW2, SW3, SW4, SW5: SW_SPST, Button_Switch_THT:SW_PUSH_6mm, symbol Switch:SW_SPST
- RV1: value R_Potentiometer -> 10k
Connections:
- net SCL/A5 is gone; now on net I2C_SCL: J3.6 (Pin_6)
- net SDA/A4 is gone; now on net I2C_SDA: J3.5 (Pin_5)
- net +5V: now also J10.2 (Pin_2), J11.3 (Pin_3), J9.1 (Pin_1), SW1.2 (B), SW2.2 (B), SW3.2 (B), SW4.2 (B), SW5.2 (B)
- net Data: now also J11.2 (Pin_2)
- net GND: now also J10.1 (Pin_1), J11.1 (Pin_1), J9.2 (Pin_2), R2.2, R3.2, R4.2, R5.2, R6.2
- net I2C_SCL: now also J10.3 (Pin_3), J9.3 (Pin_3)
- net I2C_SDA: now also J10.4 (Pin_4), J9.4 (Pin_4)
- net at D1.2 (A): now also R1.2
- new net: R5.1, SW4.1 (A)
- new net: R2.1, SW1.1 (A)
- new net: R4.1, SW3.1 (A)
- new net: R6.1, SW5.1 (A)
- new net: R3.1, SW2.1 (A)
- no-connect marks 1 -> 19
Other:
- note added: "BUTTONS"
- note added: "LED SCREEN"
- note added: "LED_light"
- note added: "MPU 6050"
- note added: "OLED SCREEN"
- note added: "TEMP SENSOR"
- note added: "UNO SHIELD"
- note added: "button_cal"
- note added: "button_light"
- note added: "button_lock"
- note added: "button_onoff"
- note added: "button_units"
- note added: "temp_sensor"
- note removed: "LED"
- note removed: "SCL/A5"
- note removed: "SDA/A4"
- company: Ali G -> (none)
- title: Uno Shield thermal pro -> (none)

Commit message: Phase_B
Connections:
- net Data is gone; now on net 7: J11.2 (Pin_2)
- net *3: now also R3.1, SW2.1 (A)
- net *5: now also R6.1, SW5.1 (A)
- net *6: now also R5.1, SW4.1 (A)
- net *9: now also R1.1
- net 2: now also R2.1, SW1.1 (A)
- net 4: now also R4.1, SW3.1 (A)
- net A0: now also RV1.2
- no-connect marks 19 -> 18
Other:
- note removed: "LED_light"
- note removed: "button_cal"
- note removed: "button_light"
- note removed: "button_lock"
- note removed: "button_onoff"
- note removed: "button_units"
- note removed: "temp_sensor"
- moved on the sheet: D1, J11, R1, R2, R3, R4, R5, R6, RV1, SW1, SW2, SW3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

Commit message: Phase_B
Other:
- note added: "DIGITAL SENSOR"
Changed lines of the file:
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@@
 	)
 	(no_connect
-		(at 119.38 41.91)
-	)
-	(no_connect
-		(at 82.55 81.28)
-	)
-	(no_connect
-		(at 82.55 53.34)
-	)
-	(no_connect
-		(at 27.94 73.66)
-	)
-	(no_connect
-		(at 82.55 48.26)
-	)
-	(no_connect
-		(at 27.94 71.12)
-	)
-	(no_connect
-		(at 27.94 76.2)
-	)
-	(no_connect
-		(at 119.38 44.45)
+		(at 120.65 43.18)
+	)
+	(no_connect
+		(at 82.55 82.55)
+	)
+	(no_connect
+		(at 82.55 54.61)
+	)
+	(no_connect
+		(at 29.21 74.93)
+	)
+	(no_connect
+		(at 82.55 49.53)
+	)
+	(no_connect
+		(at 29.21 72.39)
+	)
+	(no_connect
+		(at 29.21 77.47)
+	)
+	(no_connect
+		(at 120.65 45.72)
 	)
 	(no_connect
@@
 	)
 	(no_connect
-		(at 82.55 40.64)
-	)
-	(no_connect
-		(at 119.38 39.37)
-	)
-	(no_connect
-		(at 27.94 66.04)
-	)
-	(no_connect
-		(at 82.55 43.18)
-	)
-	(no_connect
-		(at 82.55 45.72)
-	)
-	(no_connect
-		(at 119.38 36.83)
-	)
-	(no_connect
-		(at 82.55 35.56)
-	)
-	(no_connect
-		(at 82.55 78.74)
-	)
-	(no_connect
-		(at 27.94 68.58)
+		(at 82.55 41.91)
+	)
+	(no_connect
+		(at 120.65 40.64)
+	)
+	(no_connect
+		(at 29.21 67.31)
+	)
+	(no_connect
+		(at 82.55 44.45)
+	)
+	(no_connect
+		(at 82.55 46.99)
+	)
+	(no_connect
+		(at 120.65 38.1)
+	)
+	(no_connect
+		(at 82.55 36.83)
+	)
+	(no_connect
+		(at 82.55 80.01)
+	)
+	(no_connect
+		(at 29.21 69.85)
 	)
 	(wire
@@
 			)
 		)
+	)
+	(text "DIGITAL SENSOR"
+		(exclude_from_sim no)
+		(at 149.098 93.472 0)
+		(effects
+			(font
+				(size 1.27 1.27)
+				(thickness 0.254)
+				(bold yes)
+			)
+		)

Commit message: Phase_B
Other:
- title: (none) -> Arduino Uno Temp Sensor Shield
Changed lines of the file:
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@@
 	(paper "A4")
 	(title_block
+		(title "Arduino Uno Temp Sensor Shield")
 		(date "mar. 31 mars 2015")
+		(rev "V1.0")
 	)
 	(junction
