File: Phase_B/Arduino_uno_Shield/Arduino_uno_Shield.kicad_pcb (KiCad board)
At the start: 2 copper layers, 68.6 x 53.3 mm, 20 parts, among them J1 Power, J10 CONN_DISPLAY, J11 Temp_Digital, J2 Digital/PWM, J3 Analog, J4 Digital/PWM, J9 CONN_GYRO, SW1 SW_SPST, SW2 SW_SPST, SW3 SW_SPST, SW4 SW_SPST, SW5 SW_SPST

Commit message: Phase_B
Connections:
- J11 pad 2: /Data -> /7
- R1 pad 1: unconnected-(R1-Pad1) -> /*9
- R2 pad 1: Net-(SW1-A) -> /2
- R3 pad 1: Net-(SW2-A) -> /*3
- R4 pad 1: Net-(SW3-A) -> /4
- R5 pad 1: Net-(SW4-A) -> /*6
- R6 pad 1: Net-(SW5-A) -> /*5
- RV1 pad 2: unconnected-(RV1-Pad2) -> /A0
- SW1 pad 1: Net-(SW1-A) -> /2
- SW2 pad 1: Net-(SW2-A) -> /*3
- SW3 pad 1: Net-(SW3-A) -> /4
- SW4 pad 1: Net-(SW4-A) -> /*6
- SW5 pad 1: Net-(SW5-A) -> /*5
Routing:
- net GND: track 0.00 -> 146.9 mm, vias 0 -> 3
- net +5V: track 0.00 -> 146.7 mm, vias 0 -> 3
- net /I2C_SCL: track 0.00 -> 88.9 mm, vias 0 -> 2
- net /*5: track 0.00 -> 84.4 mm
- net /I2C_SDA: track 0.00 -> 82.2 mm, vias 0 -> 1
- net /2: track 0.00 -> 63.2 mm, vias 0 -> 3
- net /*6: track 0.00 -> 55.1 mm, vias 0 -> 1
- net /4: track 0.00 -> 34.0 mm, vias 0 -> 1
- net /*3: track 0.00 -> 32.0 mm
- net /*9: track 0.00 -> 18.2 mm, vias 0 -> 1
- net /A0: track 0.00 -> 17.8 mm
- net /7: track 0.00 -> 16.1 mm
- net Net-(D1-A): track 0.00 -> 12.4 mm
- added copper zone on B.Cu, net GND

Commit message: Phase_B
Routing:
- net /I2C_SDA: track 82.2 -> 88.1 mm
- net /I2C_SCL: track 88.9 -> 93.1 mm
- net +5V: track 146.7 -> 144.5 mm
- net Net-(D1-A): track 12.4 -> 14.2 mm
- net /A0: track 17.8 -> 19.2 mm
- net GND: track 146.9 -> 147.5 mm
Other:
- board text added: "Cal"
- board text added: "Light"
- board text added: "Lock"
- board text added: "MPU6050"
- board text added: "Screen"
- board text added: "Sensor1"
- board text added: "Sensor2"
- board text added: "Units"
- board text added: "V1.0 02042025 Ali Alalwia"
- board text added: "on/off"

Commit message: Phase_B
Other:
- board text added: "Arduino UNO Temp Sensor V1.0 Ali Alalwia 02042025"
- board text removed: "V1.0 02042025 Ali Alalwia"
Changed lines of the file:
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@@
 		(grid_origin 100 100)
 		(pcbplotparams
-			(layerselection 0x0000030_ffffffff)
-			(plot_on_all_layers_selection 0x00000f0_80000001)
+			(layerselection 0x00010fc_ffffffff)
+			(plot_on_all_layers_selection 0x0000080_00000000)
 			(disableapertmacros no)
 			(usegerberextensions no)
@@
 		(tags "Through hole socket strip THT 1x08 2.54mm single row")
 		(property "Reference" "J9"
-			(at 3 9.62 180)
+			(at 0.5 -3.38 180)
 			(layer "F.SilkS")
 			(effects
@@
 		(tags "LED")
 		(property "Reference" "D1"
-			(at 0.54 5.5 90)
+			(at -1.46 -4.5 90)
 			(layer "F.SilkS")
 			(effects
@@
 		)
 	)
-	(gr_text "V1.0\n02042025\nAli Alalwia"
-		(at 102 99 0)
+	(gr_text "Arduino UNO Temp Sensor V1.0\nAli Alalwia 02042025\n\n"
+		(at 101 99.5 0)
 		(layer "F.SilkS")
 		(effects

Commit message: Phase_B
Routing:
- net GND: track 147.5 -> 81.9 mm, vias 3 -> 1
- net +5V: track 144.5 -> 158.5 mm, vias 3 -> 4
- net /4: track 34.0 -> 35.5 mm, vias 1 -> 4
- net /*6: track 55.4 -> 56.2 mm, vias 1 -> 5
