File: final_project/weather_baloon/weather_baloon.kicad_pcb (KiCad board)
At the start: 2 copper layers, 73 x 56 mm, 20 parts, among them J1 Temp_Digital, J2 Temp_Digital, J3 DHT11_Humidity, U3 40PC015G

Commit message: final_project
Parts:
- removed ADXL1: Conn_01x06, Connector_PinHeader_2.54mm:PinHeader_1x06_P2.54mm_Vertical
- added J9: CONN_GYRO, Connector_PinSocket_2.54mm:PinSocket_1x08_P2.54mm_Vertical, F.Cu at (179.5, 99.0)
- J3: footprint Connector_PinSocket_2.54mm:PinSocket_1x03_P2.54mm_Vertical -> Connector_PinSocket_2.54mm:PinSocket_1x04_P2.54mm_Vertical
- moved J3 7.11 mm to (176.5, 77.1), turned to 0 degrees
- moved OPEN_LOG1 2.18 mm to (196.3, 94.0), turned to -90 degrees
Connections:
- A1 pad 23: /ACCELEROMETER_X -> /I2C_SDA
- A1 pad 24: /ACCELEROMETER_Y -> /I2C_SCL
- A1 pad 25: unconnected-(A1-A6-Pad25) -> /ACCELEROMETER_X
- A1 pad 26: unconnected-(A1-A7-Pad26) -> /ACCELEROMETER_Y
- J3 pad 3: GND -> unconnected-(J3-Pin_3-Pad3)
Routing:
- net GND: track 104.4 -> 66.5 mm, vias 2 -> 0
- net /I2C_SDA: track 0.00 -> 37.3 mm, vias 0 -> 1
- net /I2C_SCL: track 0.00 -> 31.5 mm
- net /ACCELEROMETER_X: track 19.5 -> 0.00 mm
- net /ACCELEROMETER_Y: track 18.8 -> 0.00 mm, vias 1 -> 0
- net +5V: track 119.0 -> 135.6 mm
- net /OPEN_LOG: track 22.1 -> 37.5 mm, vias 1 -> 2
- net +3V3: track 13.4 -> 0.00 mm
- net /HUMIDITY_SENSOR: track 30.6 -> 27.9 mm
Other:
- board size 73 x 56 mm -> 70 x 56 mm
- board text added: "Blue1"
- board text added: "GYRO"
- board text added: "Green"
- board text added: "LED_Blue2"
- board text added: "LED_Orange"
- board text added: "Pressure"
- board text added: "Red"
- board text added: "Temp1"
- board text added: "Temp2"
- board text added: "Yellow"
