File: final_project/weather_baloon/weather_baloon.kicad_pcb (KiCad board)
At the start: 2 copper layers, 70 x 56 mm, 20 parts, among them J1 Temp_Digital, J2 Temp_Digital, J3 DHT11_Humidity, J9 CONN_GYRO, U3 40PC015G

Commit message: final_project
Parts:
- added J4: Conn_01x02, Connector_JST:JST_XH_B2B-XH-A_1x02_P2.50mm_Vertical, F.Cu at (172.0, 107.5)
- moved J2 15.1 mm to (175.0, 92.0)
Connections:
- A1 pad 25: /ACCELEROMETER_X -> unconnected-(A1-A6-Pad25)
- A1 pad 26: /ACCELEROMETER_Y -> unconnected-(A1-A7-Pad26)
- A1 pad 4: unconnected-(A1-GND-Pad4) -> GND
Routing:
- net VCC: track 0.00 -> 30.3 mm
- net /TEMP2: track 48.4 -> 30.6 mm
- net +5V: track 135.6 -> 118.0 mm
- net GND: track 66.5 -> 83.9 mm
- net /HUMIDITY_SENSOR: track 27.9 -> 26.8 mm
Other:
- board text added: "POWER"

Commit message: final_project
Routing:
- net GND: track 83.9 -> 7.77 mm
- net /PRESSURE_SENSOR: track 34.2 -> 24.6 mm, vias 1 -> 0
- net +5V: track 118.0 -> 110.1 mm
- net VCC: track 30.3 -> 37.3 mm
- net Net-(D6-K): track 11.6 -> 18.0 mm, vias 1 -> 0
- net /YELLOW_LED: track 17.9 -> 15.2 mm, vias 1 -> 0
- net /ORANGE_LED: track 17.4 -> 15.3 mm, vias 1 -> 0
- net Net-(D3-K): track 13.5 -> 11.8 mm, vias 1 -> 0
- net /OPEN_LOG: track 37.5 -> 37.4 mm, vias 2 -> 0
