File: final_project/weather_baloon/weather_baloon.kicad_sch (KiCad schematic)
At the start: 19 parts, among them U1 TMP36GT9, U2 TMP36GT9, U3 40PC015G, U4 CHT11, U5 DEV-13712

Commit message: finl_project
Parts:
- removed ADXL1: ~, symbol New_Library:ADXL335
- removed U1, U2: TMP36GT9, MyLibrary:XDCR_TMP36GT9, symbol TMP36GT9:TMP36GT9
- removed U4: CHT11, Connector_PinSocket_2.54mm:PinSocket_1x03_P2.54mm_Vertical, symbol Sensor:CHT11
- removed U5: DEV-13712, MyLibrary:MODULE_DEV-13712, symbol New_Library:DEV-13712
- added ADXL1, OPEN_LOG1: Conn_01x06, Connector_PinHeader_2.54mm:PinHeader_1x06_P2.54mm_Vertical, symbol Connector_Generic:Conn_01x06
- added J1: Temp_Digital, Connector_JST:JST_XH_B3B-XH-A_1x03_P2.50mm_Vertical, symbol Connector_Generic:Conn_01x03
- added J2: Temp_Digital, My_Library1:XDCR_TMP36GT9, symbol Connector_Generic:Conn_01x03
- added J3: DHT11_Humidity, Connector_PinSocket_2.54mm:PinSocket_1x03_P2.54mm_Vertical, symbol Connector_Generic:Conn_01x03
- added R7: 4.7K, Resistor_THT:R_Axial_DIN0207_L6.3mm_D2.5mm_P10.16mm_Horizontal, symbol Device:R
- D4, D5: footprint LED_THT:LED_D5.0mm -> Connector_PinSocket_2.54mm:PinSocket_1x02_P2.54mm_Vertical
- R1, R2, R3, R4, R5, R6: value R -> 1K; footprint (none) -> Resistor_THT:R_Axial_DIN0207_L6.3mm_D2.5mm_P10.16mm_Horizontal
- U3: footprint MyLibrary:DIP1330W46P254L1000H544Q8 -> My_Library1:DIP1330W46P254L1000H544Q8
Connections:
- net GND: now also ADXL1.5 (Pin_5), J1.1 (Pin_1), J2.1 (Pin_1), J3.3 (Pin_3), OPEN_LOG1.2 (Pin_2)
- net OPEN_LOG: now also OPEN_LOG1.5 (Pin_5)
- net VCC: now reaches A1.30 (VIN)
- net 3.3V renamed +3V3
- net +3V3: now also ADXL1.6 (Pin_6)
- net 5V renamed +5V
- net +5V: now also J1.3 (Pin_3), J2.3 (Pin_3), J3.1 (Pin_1), OPEN_LOG1.3 (Pin_3), R7.1
- net A0 renamed Temp1
- net Temp1: now also J1.2 (Pin_2), R7.2
- net A1 renamed TEMP2
- net TEMP2: now also J2.2 (Pin_2)
- net A2 renamed HUMIDITY_SENSOR
- net HUMIDITY_SENSOR: now also J3.2 (Pin_2)
- net A3 renamed PRESSURE_SENSOR
- net A4 renamed ACCELEROMETER_X
- net ACCELEROMETER_X: now also ADXL1.4 (Pin_4)
- net A5 renamed ACCELEROMETER_Y
- net ACCELEROMETER_Y: now also ADXL1.3 (Pin_3)
- no-connect marks 2 -> 17
Other:
- note added: "BLK"
- note added: "GND"
- note added: "GRN"
- note added: "RXI"
- note added: "ST"
- note added: "TX0"
- note added: "VCC"
- note added: "Z"

Commit message: final_project
Parts:
- removed ADXL1: Conn_01x06, Connector_PinHeader_2.54mm:PinHeader_1x06_P2.54mm_Vertical, symbol Connector_Generic:Conn_01x06
- removed J3: DHT11_Humidity, Connector_PinSocket_2.54mm:PinSocket_1x03_P2.54mm_Vertical, symbol Connector_Generic:Conn_01x03
- added J3: DHT11_Humidity, Connector_PinSocket_2.54mm:PinSocket_1x04_P2.54mm_Vertical, symbol Connector_Generic:Conn_01x04
- added J9: CONN_GYRO, Connector_PinSocket_2.54mm:PinSocket_1x08_P2.54mm_Vertical, symbol Connector_Generic:Conn_01x08
Connections:
- net +5V: now also J3.1 (Pin_1), J9.1 (Pin_1)
- net ACCELEROMETER_X: now also A1.25 (A6); no longer A1.23 (A4)
- net ACCELEROMETER_Y: now also A1.26 (A7); no longer A1.24 (A5)
- net GND: now also J3.4 (Pin_4), J9.2 (Pin_2)
- net HUMIDITY_SENSOR: now also J3.2 (Pin_2)
- new net I2C_SCL: A1.24 (A5), J9.3 (Pin_3)
- new net I2C_SDA: A1.23 (A4), J9.4 (Pin_4)
- no-connect marks 17 -> 20
Other:
- note removed: "ST"
- note removed: "Z"

Commit message: final_project
Parts:
- added J4: Conn_01x02, Connector_JST:JST_XH_B2B-XH-A_1x02_P2.50mm_Vertical, symbol Connector_Generic:Conn_01x02
Connections:
- net GND: now also A1.4 (GND), J4.1 (Pin_1)
- net VCC: now also J4.2 (Pin_2)
- net ACCELEROMETER_X: no longer names the net of A1.25 (A6)
- net ACCELEROMETER_Y: no longer names the net of A1.26 (A7)
Other:
- note added: "POWER"
